File: schematic.sch (EAGLE design)
At the start: 30 parts, among them IC1 ATMEGA168-20P, IC2 7805T, IC3 REG1117

Commit message: Fixed some things in schematic and started working on layout
Parts:
- JP4, JP8: device adafruit:PINHD-1X6 -> adafruit:PINHD-1X6B
Connections:
- new net N$4: JP3.5, JP9.5
- net +5V: no longer JP3.5, JP9.5
Changed lines of the file:
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@@
 <part name="JP2" library="adafruit" deviceset="PINHD-1X8" device="BIG"/>
 <part name="JP3" library="adafruit" deviceset="PINHD-1X8" device="BIG"/>
-<part name="JP4" library="adafruit" deviceset="PINHD-1X6" device=""/>
+<part name="JP4" library="adafruit" deviceset="PINHD-1X6" device="B"/>
 <part name="IC2" library="adafruit" deviceset="78*" device="T" technology="05"/>
 <part name="IC3" library="burr-brown" deviceset="REG1117" device=""/>
@@
 <part name="JP6" library="adafruit" deviceset="PINHD-1X8" device="BIG"/>
 <part name="JP7" library="adafruit" deviceset="PINHD-1X8" device="BIG"/>
-<part name="JP8" library="adafruit" deviceset="PINHD-1X6" device=""/>
+<part name="JP8" library="adafruit" deviceset="PINHD-1X6" device="B"/>
 <part name="JP9" library="adafruit" deviceset="PINHD-1X8" device="BIG"/>
 <part name="P+8" library="supply1" deviceset="VCC" device=""/>
@@
 <wire x1="-35.56" y1="33.02" x2="-35.56" y2="35.56" width="0.1524" layer="91"/>
 </segment>
-<segment>
-<pinref part="P+6" gate="1" pin="+5V"/>
-<wire x1="-12.7" y1="78.74" x2="-12.7" y2="71.12" width="0.1524" layer="91"/>
-<pinref part="JP3" gate="G$1" pin="5"/>
-<wire x1="-12.7" y1="71.12" x2="-30.48" y2="71.12" width="0.1524" layer="91"/>
-<pinref part="JP9" gate="G$1" pin="5"/>
-<wire x1="-40.64" y1="71.12" x2="-30.48" y2="71.12" width="0.1524" layer="91"/>
-<junction x="-30.48" y="71.12"/>
-</segment>
 </net>
 <net name="+3V3" class="0">
@@
 <wire x1="-91.44" y1="55.88" x2="-91.44" y2="83.82" width="0.1524" layer="91"/>
 <junction x="-91.44" y="83.82"/>
-<label x="-99.06" y="83.82" size="1.778" layer="95" rot="R90" xref="yes"/>
 </segment>
 </net>
@@
 </segment>
 </net>
+<net name="N$4" class="0">
+<segment>
+<pinref part="JP3" gate="G$1" pin="5"/>
+<wire x1="-12.7" y1="71.12" x2="-30.48" y2="71.12" width="0.1524" layer="91"/>
+<pinref part="JP9" gate="G$1" pin="5"/>
+<wire x1="-40.64" y1="71.12" x2="-30.48" y2="71.12" width="0.1524" layer="91"/>
+<junction x="-30.48" y="71.12"/>
+</segment>
+</net>

Commit message: Finished layout, still needs cleaning
Parts:
- JP3: device adafruit:PINHD-1X8BIG -> adafruit:PINHD-1X6B
- LED1, LED2: device adafruit:LED5MM -> adafruit:LED3MM
Connections:
- removed net N$4: JP3.5, JP9.5
- net +3V3: now also JP3.2; no longer JP3.4
- net +5V: now also JP3.3, JP9.5
- net GND: now also JP3.4, JP3.5; no longer JP3.6, JP3.7
- net RESET: now also JP3.1; no longer JP3.3
- net VIN: now also JP3.6; no longer JP3.8
Changed lines of the file:
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@@
 <part name="JP1" library="adafruit" deviceset="PINHD-1X8" device="BIG"/>
 <part name="JP2" library="adafruit" deviceset="PINHD-1X8" device="BIG"/>
-<part name="JP3" library="adafruit" deviceset="PINHD-1X8" device="BIG"/>
 <part name="JP4" library="adafruit" deviceset="PINHD-1X6" device="B"/>
 <part name="IC2" library="adafruit" deviceset="78*" device="T" technology="05"/>
@@
 <part name="R2" library="rcl" deviceset="R-EU_" device="0207/7"/>
 <part name="P+10" library="supply1" deviceset="VCC" device=""/>
-<part name="LED1" library="adafruit" deviceset="LED" device="5MM"/>
+<part name="LED1" library="adafruit" deviceset="LED" device="3MM"/>
 <part name="GND14" library="supply1" deviceset="GND" device=""/>
 <part name="R3" library="rcl" deviceset="R-EU_" device="0207/7"/>
-<part name="LED2" library="adafruit" deviceset="LED" device="5MM"/>
+<part name="LED2" library="adafruit" deviceset="LED" device="3MM"/>
 <part name="GND15" library="supply1" deviceset="GND" device=""/>
+<part name="JP3" library="adafruit" deviceset="PINHD-1X6" device="B"/>
 </parts>
 <sheets>
@@
 <instance part="JP1" gate="G$1" x="111.76" y="50.8"/>
 <instance part="JP2" gate="G$1" x="111.76" y="27.94"/>
-<instance part="JP3" gate="G$1" x="-33.02" y="73.66" rot="MR0"/>
 <instance part="JP4" gate="A" x="111.76" y="76.2"/>
 <instance part="IC2" gate="A1" x="-76.2" y="83.82"/>
@@
 <instance part="LED2" gate="G$1" x="-93.98" y="15.24"/>
 <instance part="GND15" gate="1" x="-93.98" y="5.08"/>
+<instance part="JP3" gate="A" x="-33.02" y="68.58" rot="MR0"/>
 </instances>
 <busses>
@@
 </segment>
 <segment>
-<pinref part="JP3" gate="G$1" pin="7"/>
-<wire x1="-30.48" y1="66.04" x2="-22.86" y2="66.04" width="0.1524" layer="91"/>
 <wire x1="-22.86" y1="66.04" x2="-22.86" y2="68.58" width="0.1524" layer="91"/>
-<pinref part="JP3" gate="G$1" pin="6"/>
-<wire x1="-22.86" y1="68.58" x2="-30.48" y2="68.58" width="0.1524" layer="91"/>
 <wire x1="-22.86" y1="68.58" x2="-12.7" y2="68.58" width="0.1524" layer="91"/>
-<junction x="-22.86" y="68.58"/>
 <wire x1="-12.7" y1="68.58" x2="-12.7" y2="60.96" width="0.1524" layer="91"/>
 <pinref part="GND7" gate="1" pin="GND"/>
 <pinref part="JP9" gate="G$1" pin="7"/>
+<pinref part="JP3" gate="A" pin="5"/>
 <wire x1="-40.64" y1="66.04" x2="-30.48" y2="66.04" width="0.1524" layer="91"/>
+<pinref part="JP9" gate="G$1" pin="6"/>
+<pinref part="JP3" gate="A" pin="4"/>
+<wire x1="-40.64" y1="68.58" x2="-30.48" y2="68.58" width="0.1524" layer="91"/>
+<wire x1="-30.48" y1="66.04" x2="-30.48" y2="68.58" width="0.1524" layer="91"/>
 <junction x="-30.48" y="66.04"/>
-<pinref part="JP9" gate="G$1" pin="6"/>
-<wire x1="-30.48" y1="68.58" x2="-40.64" y2="68.58" width="0.1524" layer="91"/>
 <junction x="-30.48" y="68.58"/>
+<wire x1="-30.48" y1="66.04" x2="-22.86" y2="66.04" width="0.1524" layer="91"/>
 </segment>
 <segment>
@@
 <wire x1="-35.56" y1="33.02" x2="-35.56" y2="35.56" width="0.1524" layer="91"/>
 </segment>
+<segment>
+<pinref part="P+6" gate="1" pin="+5V"/>
+<wire x1="-12.7" y1="78.74" x2="-12.7" y2="71.12" width="0.1524" layer="91"/>
+<pinref part="JP9" gate="G$1" pin="5"/>
+<pinref part="JP3" gate="A" pin="3"/>
+<wire x1="-40.64" y1="71.12" x2="-30.48" y2="71.12" width="0.1524" layer="91"/>
+<wire x1="-12.7" y1="71.12" x2="-30.48" y2="71.12" width="0.1524" layer="91"/>
+<junction x="-30.48" y="71.12"/>
+</segment>
 </net>
 <net name="+3V3" class="0">
@@
 </segment>
 <segment>
-<pinref part="JP3" gate="G$1" pin="4"/>
 <pinref part="+3V3" gate="G$1" pin="+3V3"/>
-<wire x1="-30.48" y1="73.66" x2="-17.78" y2="73.66" width="0.1524" layer="91"/>
 <wire x1="-17.78" y1="73.66" x2="-17.78" y2="78.74" width="0.1524" layer="91"/>
 <pinref part="JP9" gate="G$1" pin="4"/>
-<wire x1="-30.48" y1="73.66" x2="-40.64" y2="73.66" width="0.1524" layer="91"/>
+<pinref part="JP3" gate="A" pin="2"/>
+<wire x1="-40.64" y1="73.66" x2="-30.48" y2="73.66" width="0.1524" layer="91"/>
+<wire x1="-30.48" y1="73.66" x2="-17.78" y2="73.66" width="0.1524" layer="91"/>
 <junction x="-30.48" y="73.66"/>
 </segment>
@@
 </segment>
 <segment>
-<pinref part="JP3" gate="G$1" pin="3"/>
-<wire x1="-30.48" y1="76.2" x2="-22.86" y2="76.2" width="0.1524" layer="91"/>
 <wire x1="-22.86" y1="76.2" x2="-22.86" y2="88.9" width="0.1524" layer="91"/>
 <wire x1="-22.86" y1="88.9" x2="-20.32" y2="88.9" width="0.1524" layer="91"/>
 <label x="-20.32" y="88.9" size="1.778" layer="95" xref="yes"/>
 <pinref part="JP9" gate="G$1" pin="3"/>
+<pinref part="JP3" gate="A" pin="1"/>
 <wire x1="-40.64" y1="76.2" x2="-30.48" y2="76.2" width="0.1524" layer="91"/>
+<wire x1="-30.48" y1="76.2" x2="-22.86" y2="76.2" width="0.1524" layer="91"/>
 <junction x="-30.48" y="76.2"/>
 </segment>
@@
 </segment>
 <segment>
-<pinref part="JP3" gate="G$1" pin="8"/>
+<pinref part="JP9" gate="G$1" pin="8"/>
+<pinref part="JP3" gate="A" pin="6"/>
+<wire x1="-40.64" y1="63.5" x2="-30.48" y2="63.5" width="0.1524" layer="91"/>
 <wire x1="-30.48" y1="63.5" x2="-22.86" y2="63.5" width="0.1524" layer="91"/>
+<junction x="-30.48" y="63.5"/>
 <label x="-22.86" y="63.5" size="1.778" layer="95" xref="yes"/>
-<pinref part="JP9" gate="G$1" pin="8"/>
-<wire x1="-30.48" y1="63.5" x2="-40.64" y2="63.5" width="0.1524" layer="91"/>
-<junction x="-30.48" y="63.5"/>
-</segment>
-</net>
-<net name="N$4" class="0">
-<segment>
-<pinref part="JP3" gate="G$1" pin="5"/>
-<wire x1="-12.7" y1="71.12" x2="-30.48" y2="71.12" width="0.1524" layer="91"/>
-<pinref part="JP9" gate="G$1" pin="5"/>
-<wire x1="-40.64" y1="71.12" x2="-30.48" y2="71.12" width="0.1524" layer="91"/>
-<junction x="-30.48" y="71.12"/>
-</segment>
-</net>
+</segment>
+</net>

Commit message: First version
Parts:
- removed Q1: (no value), adafruit:CRYSTALHC49S
- added XTAL: 16M, adafruit:CRYSTALHC49S
- C1, C7: value (none) -> 100nF
- C2, C3: value (none) -> 22pF
- C4, C5: value (none) -> 10uF
- C6: value (none) -> 47uF
- R1: value (none) -> 10k
- R2, R3: value (none) -> 1k
- renumbered IC1 to ATMEGA, IC2 to REG5, IC3 to REG33, ISP1 to ISP, JP10 to SERIAL, JP5 to 3.3-5V, LED1 to POWER, LED2 to LED13, S1 to RESET, U$1 to IN
Connections:
- net N$2: now also XTAL.2; no longer Q1.2
- net N$3: now also XTAL.1; no longer Q1.1
Other:
- moved on the sheet: C2, C3
