File: Suino board.brd (EAGLE design)
At the start: 100 x 80 mm, 30 parts

Commit message: Added frame and name
Parts:
- moved C1 4.58 mm to (59.7, 39.4), turned to 90 degrees
- moved C2 1.27 mm to (52.1, 38.1), turned to 90 degrees
- turned C3 to 90 degrees
Routing:
- net VCC: track 157.1 -> 149.0 mm
- net GND: track 275.7 -> 269.0 mm
- net N$2: track 11.7 -> 9.94 mm
- net N$3: track 10.8 -> 9.60 mm
- net RESET: track 136.7 -> 137.4 mm
