File: Suino board.sch (EAGLE design)
At the start: 30 parts

Commit message: Added frame and name
Other:
- note added: "Robson Couto"
- note added: "github.com/dragaosemchama"
- note added: "github.com/robsoncouto"
- note added: "www.dragaosemchama.com.br"
- moved on the sheet: 3.3-5V, C1, C4, C5, C6, D1, IN, JP3, JP9, LED13, POWER, R2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
